File: hp3478a-ch32-ext.kicad_pcb (KiCad board)
At the start: 4 copper layers, 32.5 x 50 mm, 26 parts, among them J1 Conn_GPIB, J2 Pwr, J3 Debug, Q1 BSS138, U1 CH32V003FxUx, U2 TLV76701DRVx

Commit message: chore: _
Parts:
- removed U1: CH32V003FxUx, Package_DFN_QFN:QFN-20-1EP_3x3mm_P0.4mm_EP1.65x1.65mm_ThermalVias
- added C4: 100n, Capacitor_SMD:C_0402_1005Metric, F.Cu at (61.5, 62.6)
- added C5: 100n, Capacitor_SMD:C_0402_1005Metric, F.Cu at (52.8, 59.5)
- added C6: 100n, Capacitor_SMD:C_0402_1005Metric, F.Cu at (56.1, 51.2)
- added C7: 100n, Capacitor_SMD:C_0402_1005Metric, F.Cu at (64.5, 56.0)
- added C8: 100n, Capacitor_SMD:C_0402_1005Metric, F.Cu at (79.9, 62.7)
- added D8: USBLC6-2SC6, PCM_Package_TO_SOT_SMD_AKL:SOT-23-6, F.Cu at (83.9, 61.0)
- added J4: USB, Connector_Molex:Molex_PicoBlade_53047-0410_1x04_P1.25mm_Vertical, F.Cu at (81.0, 51.7)
- added SW1: RST, Button_Switch_SMD:SW_SPST_PTS810, F.Cu at (84.7, 56.2)
- added U3: CH32V203CxTx, Package_QFP:LQFP-48_7x7mm_P0.5mm, F.Cu at (58.6, 57.0)
- C1, C2: value 10uF -> 10u
- C3: value 100nF -> 100n
- moved D7 40.0 mm to (103.0, 53.1)
- moved D2 40.0 mm to (98.3, 48.3)
- moved D3 40.0 mm to (98.3, 51.8)
- moved D5 40.0 mm to (97.8, 61.7)
- moved D6 40.0 mm to (100.3, 69.0)
- moved D4 20.2 mm to (73.7, 68.7)
- moved RN2 5.50 mm to (54.0, 65.0)
- moved D1 3.81 mm to (51.9, 82.5), turned to 0 degrees
- moved C3 3.78 mm to (64.5, 58.5), turned to 90 degrees
- moved RN3 3.10 mm to (58.0, 68.0)
- moved Q1 1.82 mm to (52.0, 79.7)
- moved RN1 1.40 mm to (54.0, 48.0)
- moved RN4 0.92 mm to (63.6, 65.3)
Connections:
- BZ1 pad 1: +5V -> VDD
- C2 pad 1: +5V -> VDD
- C3 pad 1: +5V -> VDD
- D1 pad 1: +5V -> VDD
- J3 pad 1: +5V -> VDD
- R1 pad 1: +5V -> VDD
- U2 pad 1: +5V -> VDD
Routing:
- net +5V: track 69.3 -> 0.00 mm, vias 2 -> 0
- net /SWIO: track 35.7 -> 0.00 mm, vias 2 -> 0
- net GND: track 34.3 -> 5.21 mm, vias 62 -> 0
- net /BUZZ: track 21.7 -> 0.00 mm, vias 2 -> 0
- net /REN: track 16.9 -> 0.00 mm
- net /DIO7: track 15.8 -> 0.00 mm
- net /DIO8: track 15.6 -> 0.00 mm
- net /DIO6: track 14.5 -> 0.00 mm
- net /DIO5: track 13.0 -> 0.00 mm
- net /ATN: track 11.5 -> 0.00 mm
- net Net-(BZ1--): track 10.9 -> 0.00 mm
- net /SRQ: track 10.8 -> 0.00 mm
- net /IFC: track 9.92 -> 0.00 mm, vias 2 -> 0
- net /NDAC: track 9.84 -> 0.00 mm
- net VDD: track 0.00 -> 7.21 mm
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Other:
- board size 32.5 x 50 mm -> 40 x 50 mm

Commit message: chore: _
Parts:
- added C10: 100n, Capacitor_SMD:C_0402_1005Metric, F.Cu at (51.2, 73.4)
- added C11: ~10pF, Capacitor_SMD:C_0402_1005Metric, F.Cu at (60.3, 60.3)
- added C12: ~10pF, Capacitor_SMD:C_0402_1005Metric, F.Cu at (54.9, 60.4)
- added C9: 100n, Capacitor_SMD:C_0402_1005Metric, F.Cu at (52.1, 86.1)
- added J5: Micro_SD_Card_Det1, Miiine:J_SD_Card-micro_socket_A, B.Cu at (50.0, 80.3)
- added R10: 47k, Resistor_SMD:R_0402_1005Metric, F.Cu at (47.8, 76.4)
- added R5: 47k, Resistor_SMD:R_0402_1005Metric, F.Cu at (49.1, 76.4)
- added R6: 47k, Resistor_SMD:R_0402_1005Metric, F.Cu at (50.4, 76.4)
- added R7: 47k, Resistor_SMD:R_0402_1005Metric, F.Cu at (51.7, 76.4)
- added R8: 47k, Resistor_SMD:R_0402_1005Metric, F.Cu at (53.0, 76.4)
- added R9: 47k, Resistor_SMD:R_0402_1005Metric, F.Cu at (54.3, 76.4)
- added U3: AHT20, Miiine:AHT20, F.Cu at (49.8, 85.6)
- added Y1: 24MHz, 10pF, Crystal:Crystal_SMD_3225-4Pin_3.2x2.5mm, F.Cu at (57.6, 60.4)
- moved D8 53.4 mm to (34.4, 81.2), turned to 180 degrees
- moved J4 51.7 mm to (39.3, 82.2), turned to -90 degrees
- moved SW1 42.4 mm to (49.8, 80.3)
- moved C8 32.0 mm to (53.2, 80.4), turned to -90 degrees
- moved D7 19.5 mm to (83.8, 57.2)
- moved D2 19.5 mm to (79.2, 52.4)
- moved D3 19.5 mm to (79.2, 55.9)
- moved D5 19.5 mm to (78.8, 65.8)
- moved D6 19.5 mm to (81.2, 73.1)
- moved J3 16.1 mm to (29.9, 85.7)
- moved C5 14.1 mm to (57.0, 46.0), turned to 0 degrees
- moved C4 11.4 mm to (53.0, 55.0), turned to 90 degrees
- moved C3 9.35 mm to (55.1, 57.9), turned to 180 degrees
- moved J2 9.02 mm to (30.1, 73.0)
- moved C1 8.68 mm to (33.2, 74.4)
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- renumbered U3 to U1
Connections:
- D8 pad 1: /USB_IN_D_N -> /USB_IN_D_P
- D8 pad 3: /USB_IN_D_P -> /USB_IN_D_N
- D8 pad 4: /USB_D_P -> /USBFS_DN
- D8 pad 6: /USB_D_N -> /USBFS_DP
- J2 pad 2: +5V -> VDD
- U1 pad 10: unconnected-(U3-PA0-Pad10) -> /I2C_SCL
- U1 pad 11: unconnected-(U3-PA1-Pad11) -> /I2C_SDA
- U1 pad 14: unconnected-(U3-PA4-Pad14) -> /SPI1_NSS
- U1 pad 15: unconnected-(U3-PA5-Pad15) -> /SPI1_SCK
- U1 pad 16: unconnected-(U3-PA6-Pad16) -> /SPI1_MISO
- U1 pad 17: unconnected-(U3-PA7-Pad17) -> /SPI1_MOSI
- U1 pad 2: unconnected-(U3-PC13-Pad2) -> /BUZZ
- U1 pad 32: /USB_D_N -> /NDAC
- U1 pad 33: /USB_D_P -> /NRFD
- U1 pad 38: /NDAC -> /DAV
- U1 pad 39: /NRFD -> /EOI
- U1 pad 40: /DAV -> /DIO4
- U1 pad 41: /EOI -> /DIO3
- U1 pad 42: /DIO4 -> /USBFS_DN
- U1 pad 43: /DIO3 -> /USBFS_DP
- U1 pad 5: unconnected-(U3-OSC_IN-Pad5) -> Net-(U1-OSC_IN)
- U1 pad 6: unconnected-(U3-OSC_OUT-Pad6) -> Net-(U1-OSC_OUT)
Routing:
- net Net-(J1-NRFD): track 8.97 -> 0.00 mm, vias 1 -> 0
- net Net-(J1-DIO1): track 8.40 -> 0.00 mm
- net Net-(J1-DIO5): track 7.88 -> 0.00 mm
- net Net-(J1-DIO2): track 7.75 -> 0.00 mm
- net Net-(J1-DAV): track 7.35 -> 0.00 mm
- net VDD: track 7.21 -> 0.00 mm
- net Net-(J1-DIO3): track 7.06 -> 0.00 mm
- net /DIO2: track 6.91 -> 0.00 mm
- net /DIO3: track 6.82 -> 0.00 mm
- net /DIO1: track 6.78 -> 0.00 mm
- net /DIO4: track 6.59 -> 0.00 mm
- net /EOI: track 5.61 -> 0.00 mm
- net Net-(J1-EOI): track 5.61 -> 0.00 mm
- net GND: track 5.21 -> 0.00 mm
- net Net-(J1-NDAC): track 4.83 -> 0.00 mm
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
Commit message: chore: -
Parts:
- removed J3: Debug, Connector_PinHeader_2.54mm:PinHeader_1x03_P2.54mm_Vertical
- added DEBUG: DEBUG, Connector:Tag-Connect_TC2030-IDC-NL_2x03_P1.27mm_Vertical, F.Cu at (54.2, 40.3)
- added R11: 10k, Resistor_SMD:R_0402_1005Metric, F.Cu at (34.2, 85.4)
- added R12: 10k, Resistor_SMD:R_0402_1005Metric, F.Cu at (31.5, 83.3)
- added R13: 10k, Resistor_SMD:R_0402_1005Metric, F.Cu at (53.3, 47.8)
- added R14: 10k, Resistor_SMD:R_0402_1005Metric, F.Cu at (64.2, 46.0)
- added kibuzzard-68A1C101: G***, kibuzzard-68A1C101, F.Cu at (39.1, 83.7)
- added kibuzzard-68A1C131: G***, kibuzzard-68A1C131, B.Cu at (34.7, 86.7)
- added kibuzzard-68A1C183: G***, kibuzzard-68A1C183, F.Cu at (64.2, 72.7)
- added kibuzzard-68A1C999: G***, kibuzzard-68A1C999, F.Cu at (46.2, 87.0)
- moved D6 35.3 mm to (61.0, 44.2), turned to 0 degrees
- moved D8 27.8 mm to (61.2, 73.9)
- moved J4 26.5 mm to (65.8, 80.2), turned to 90 degrees
- moved D2 23.3 mm to (57.4, 44.2)
- moved D3 23.2 mm to (57.3, 63.4)
- moved D7 20.7 mm to (63.5, 60.9)
- moved D5 18.2 mm to (60.6, 66.8)
- moved U3 17.8 mm to (32.0, 85.9)
- moved D4 17.5 mm to (57.3, 66.6), turned to 180 degrees
- moved C8 17.5 mm to (35.7, 80.2)
- moved C9 16.9 mm to (35.2, 86.4)
- moved SW1 10.7 mm to (39.1, 80.2)
- moved R4 5.85 mm to (44.7, 80.0), turned to 90 degrees
- moved R6 5.23 mm to (45.2, 75.8)
- moved R3 5.19 mm to (47.2, 77.5)
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Connections:
- C9 pad 1: Net-(U3-VDD) -> VDD
- D8 pad 1: /USB_IN_D_P -> /USB_IN_D_N
- D8 pad 3: /USB_IN_D_N -> /USB_IN_D_P
- D8 pad 4: /USBFS_DN -> /USBFS_DP
- D8 pad 6: /USBFS_DP -> /USBFS_DN
- U1 pad 13: unconnected-(U1-PA3-Pad13) -> /CARD_DET
- U3 pad 2: Net-(U3-VDD) -> VDD
Routing:
- net VDD: track 0.00 -> 141.5 mm, vias 0 -> 9
- net /nRST: track 0.00 -> 60.7 mm, vias 0 -> 5
- net GND: track 0.00 -> 60.2 mm, vias 0 -> 70
- net /I2C_SDA: track 0.00 -> 52.7 mm, vias 0 -> 2
- net /I2C_SCL: track 0.00 -> 50.5 mm, vias 0 -> 2
- net /SPI1_MOSI: track 0.00 -> 40.5 mm, vias 0 -> 2
- net /SPI1_NSS: track 0.00 -> 39.9 mm, vias 0 -> 2
- net /DIO5: track 0.00 -> 38.0 mm, vias 0 -> 2
- net /VBUS: track 0.00 -> 35.3 mm, vias 0 -> 2
- net /SPI1_MISO: track 0.00 -> 34.5 mm, vias 0 -> 2
- net /SPI1_SCK: track 0.00 -> 34.3 mm, vias 0 -> 1
- net /BUZZ: track 0.00 -> 34.1 mm, vias 0 -> 4
- net /CARD_DET: track 0.00 -> 31.2 mm, vias 0 -> 2
- net /DIO6: track 0.00 -> 29.7 mm, vias 0 -> 2
- net /USBFS_DN: track 0.00 -> 27.9 mm, vias 0 -> 2
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Other:
- board text added: "+3.3V"
- board text added: "HP 3478A Ext."
- board text removed: "+5V"
- board text removed: "HP 3478A Extension"
- board text removed: "SWD"
