File: hp3478a-ch32-ext.kicad_pcb (KiCad board)
At the start: 4 copper layers, 40 x 50 mm, 55 parts, among them J1 Conn_GPIB, J2 Pwr, J4 USB, J5 Micro_SD_Card_Det1, Q1 BSS138, SW1 RST, U1 CH32V203CxTx, U2 TLV76701DRVx, U3 AHT20, Y1 24MHz, 10pF

Commit message: chore: _
Routing:
- net GND: track 60.1 -> 61.8 mm, vias 70 -> 78
