File: hp3478a-ch32-ext.kicad_sch (KiCad schematic)
At the start: 25 parts, among them J1 Conn_GPIB, J2 Pwr, J3 Debug, Q1 BSS138, U1 CH32V003FxUx, U2 TLV76701DRVx

Commit message: chore: _
Parts:
- removed U1: CH32V003FxUx, Package_DFN_QFN:QFN-20-1EP_3x3mm_P0.4mm_EP1.65x1.65mm_ThermalVias, symbol MCU_WCH_CH32V0:CH32V003FxUx
- added C4, C5, C6, C7, C8: 100n, Capacitor_SMD:C_0402_1005Metric, symbol Device:C_Small
- added D8: USBLC6-2SC6, PCM_Package_TO_SOT_SMD_AKL:SOT-23-6, symbol PCM_Diode_TVS_AKL:USBLC6-2SC6
- added J4: USB, Connector_Molex:Molex_PicoBlade_53047-0410_1x04_P1.25mm_Vertical, symbol Connector_Generic:Conn_01x04
- added SW1: RST, Button_Switch_SMD:SW_SPST_PTS810, symbol Switch:SW_Push
- added U3: CH32V203CxTx, Package_QFP:LQFP-48_7x7mm_P0.5mm, symbol MCU_WCH_CH32V2:CH32V203CxTx
- C1, C2: value 10uF -> 10u
- C3: value 100nF -> 100n
Connections:
- net +5V: no longer BZ1.1 (+), C2.1, C3.1, D1.1 (K), J3.1 (Pin_1), R1.1, U2.1 (OUT)
- net ATN: now also U3.29 (PA8)
- net DAV: now also U3.40 (PB4)
- net DIO1: now also U3.46 (PB9)
- net DIO2: now also U3.45 (PB8)
- net DIO3: now also U3.43 (PB7)
- net DIO4: now also U3.42 (PB6)
- net DIO5: now also U3.28 (PB15)
- net DIO6: now also U3.27 (PB14)
- net DIO7: now also U3.26 (PB13)
- net DIO8: now also U3.25 (PB12)
- net EOI: now also U3.41 (PB5)
- net GND: now also C4.2, C5.2, C6.2, C7.2, C8.2, D8.2 (VN), J4.4 (Pin_4), SW1.2, U3.23 (VSS), U3.35 (VSS), U3.47 (VSS), U3.8 (VSSA)
- net IFC: now also U3.31 (PA10)
- net NDAC: now also U3.38 (PA15)
- net NRFD: now also U3.39 (PB3)
- net REN: now also U3.22 (PB11)
- net SRQ: now also U3.30 (PA9)
- new net BOOT0: U3.44 (BOOT0)
- new net BOOT1: U3.20 (PB2)
- new net SWCLK: U3.37 (SWCLK)
- new net SWDIO: U3.34 (SWDIO)
- new net USB_D_N: D8.6 (L1), U3.32 (PA11)
- new net USB_D_P: D8.4 (L2), U3.33 (PA12)
- new net USB_IN_D_N: D8.1 (L1), J4.2 (Pin_2)
- new net USB_IN_D_P: D8.3 (L2), J4.3 (Pin_3)
- new net VBUS: D8.5 (VP), J4.1 (Pin_1), U3.21 (PB10)
- new net VDD: BZ1.1 (+), C2.1, C3.1, C4.1, C5.1, C6.1, C7.1, D1.1 (K), J3.1 (Pin_1), R1.1, U2.1 (OUT), U3.1 (VBAT), U3.24 (VDD_VIO), U3.36 (VDD), U3.48 (VDD), U3.9 (VDDA)
- new net nRST: C8.1, SW1.1, U3.7 (~{RST})
Other:
- note added: "~8.5 mA clamp current D5 and D7 can be BAT54JW"
- note removed: "B5819WS ~8.5 mA clamp current"
- moved on the sheet: C3, J1, J2, J3, RN1, RN2, RN3, RN4

Commit message: chore: _
Parts:
- added C10, C9: 100n, Capacitor_SMD:C_0402_1005Metric, symbol Device:C_Small
- added C11, C12: ~10pF, Capacitor_SMD:C_0402_1005Metric, symbol Device:C_Small
- added J5: Micro_SD_Card_Det1, Miiine:J_SD_Card-micro_socket_A, symbol Connector:Micro_SD_Card_Det1
- added R10, R5, R6, R7, R8, R9: 47k, Resistor_SMD:R_0402_1005Metric, symbol Device:R_Small
- added U3: AHT20, Miiine:AHT20, symbol Mineee:AHT20
- added Y1: 24MHz, 10pF, Crystal:Crystal_SMD_3225-4Pin_3.2x2.5mm, symbol Device:Crystal_GND24_Small
- renumbered U3 to U1
Connections:
- net +5V is gone; now on net VDD: J2.2 (Pin_2)
- net BUZZ: now also U1.2 (PC13)
- net DAV: now also U1.38 (PA15); no longer U1.40 (PB4)
- net DIO3: now also U1.41 (PB5); no longer U1.43 (PB7)
- net DIO4: now also U1.40 (PB4); no longer U1.42 (PB6)
- net EOI: now also U1.39 (PB3); no longer U1.41 (PB5)
- net GND: now also C10.2, C11.2, C12.1, C9.2, J5.10 (SHIELD), J5.6 (VSS), U3.5 (GND), Y1.2, Y1.4
- net NDAC: now also U1.32 (PA11); no longer U1.38 (PA15)
- net NRFD: now also U1.33 (PA12); no longer U1.39 (PB3)
- net USB_IN_D_N: now also D8.3 (L2); no longer D8.1 (L1)
- net USB_IN_D_P: now also D8.1 (L1); no longer D8.3 (L2)
- net VDD: now also C10.1, J5.4 (VDD), R10.1, R5.1, R6.1, R7.1, R8.1, R9.1
- net I2C_SCL: now reaches U1.10 (PA0)
- net I2C_SCL: now also U3.3 (SCL)
- net I2C_SDA: now reaches U1.11 (PA1)
- net I2C_SDA: now also U3.4 (SDA)
- net SPI1_NSS: now reaches U1.14 (PA4)
- net SPI1_NSS: now also J5.2 (DAT3/CD), R5.2
- net SPI1_SCK: now reaches U1.15 (PA5)
- net SPI1_SCK: now also J5.5 (CLK)
- net SPI1_MISO: now reaches U1.16 (PA6)
- net SPI1_MISO: now also J5.7 (DAT0), R7.2
- net SPI1_MOSI: now reaches U1.17 (PA7)
- net SPI1_MOSI: now also J5.3 (CMD), R6.2
- net at U1.5 (OSC_IN): now also C12.2, Y1.1
- net at U1.6 (OSC_OUT): now also C11.1, Y1.3
- net USB_D_N renamed USBFS_DP
- net USBFS_DP: now also U1.43 (PB7); no longer U1.32 (PA11)
- net USB_D_P renamed USBFS_DN
- net USBFS_DN: now also U1.42 (PB6); no longer U1.33 (PA12)
- new net: J5.1 (DAT2), R10.2
- new net: J5.8 (DAT1), R8.2
- new net: C9.1, U3.2 (VDD)
- new net CARD_DET: J5.9 (DET), R9.2
Other:
- note added: "bitbanged i2c"
- moved on the sheet: U1

Commit message: chore: -
Parts:
- removed J3: Debug, Connector_PinHeader_2.54mm:PinHeader_1x03_P2.54mm_Vertical, symbol Connector_Generic:Conn_01x03
- added J6: DEBUG, Connector:Tag-Connect_TC2030-IDC-NL_2x03_P1.27mm_Vertical, symbol Connector:Conn_ARM_SWD_TagConnect_TC2030-NL
- added R11, R12, R13, R14: 10k, Resistor_SMD:R_0402_1005Metric, symbol Device:R_Small
Connections:
- net BOOT0: now also R13.1
- net BOOT1: now also R14.1
- net CARD_DET: now also U1.13 (PA3)
- net GND: now also J6.5 (GND), R13.2, R14.2
- net I2C_SCL: now also R11.2
- net I2C_SDA: now also R12.2
- net SWCLK: now also J6.4 (SWCLK)
- net SWDIO: now also J6.2 (SWDIO)
- net USBFS_DN: now also D8.6 (L1); no longer D8.4 (L2)
- net USBFS_DP: now also D8.4 (L2); no longer D8.6 (L1)
- net USB_IN_D_N: now also D8.1 (L1); no longer D8.3 (L2)
- net USB_IN_D_P: now also D8.3 (L2); no longer D8.1 (L1)
- net VDD: now also C9.1, U3.2 (VDD), J6.1 (VCC), R11.1, R12.1
- net nRST: now also J6.3 (~{RESET})
- no-connect marks 3 -> 7
Other:
- moved on the sheet: C3, C4, C5, C6, C7, C9, U3

Commit message: chore: upd
Parts:
- R1: value 430k -> 470k
- R2: value 82k -> 150k
Connections:
- no-connect marks 7 -> 9
Other:
- note added: "Connectors"
- note added: "ESD prot"
- note added: "Temp sense"
- note added: "~3.293V"
- company: (none) -> kuwoyuki
- title: (none) -> HP3478A Extension
- moved on the sheet: C1, C10, C11, C12, C2, C3, C4, C5, C6, C7, C8, C9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
